Commit message: Add follow-object, RL locomotion, teleop camera + project README
- quadruped_perception + quadruped_follow: camera RGBD -> YOLO -> tracker ->
  target_pose -> action track_object (PID bam muc tieu, giu stop_distance).
  Da kiem chung so lieu that trong Gazebo (robot bam toi 0.8m, bam muc tieu dong).
- quadruped_teleop: them khung camera /camera/image + bounding box tu /detections.
- quadruped_rl: chay policy ONNX (unitree-go2-velocity-flat, BSD-3) thay gait
  rule-based. obs 45 chieu -> ONNX -> PD torque (effort). Fix 3 bug: PD 2 vong,
  startup hand-off (position->effort switch), remap joint_ids_map (FR<->FL,RR<->RL).
  Robot dung + di duoc trong Gazebo (con residual drift do gap sim-to-sim).
  + mujoco_demo/: lai Go2 bang joystick trong MuJoCo (di chuan, khong drift) +
  course chuong ngai (cau thang) de test gioi han.
- quadruped_interfaces: them TrackObject.action, TrackedTarget.msg.
- quadruped_description: them camera RGBD + effort interface + target_ball;
  visual dung box primitive (mesh .dae lam hong render camera tren GPU hybrid).
- README.md du an voi hinh anh; cap nhat CLAUDE.md, TODO.md.

Co-Authored-By: Claude Opus 4.8 <noreply@anthropic.com>

File: quadruped_ws/src/quadruped_description/xacro/gazebo.xacro (robot description, xacro)
@@ -29,4 +29,27 @@
         </sensor>
     </gazebo>
+    <!-- Camera RGBD dung cho track_object (quadruped_perception) - publish
+         camera/image (mau), camera/depth_image (32FC1), camera/camera_info.
+         gz-sim-sensors-system + render_engine ogre2 da bat san trong
+         worlds/flat_ground.sdf. -->
+    <gazebo reference="camera_link">
+        <sensor name="camera_sensor" type="rgbd_camera">
+            <always_on>true</always_on>
+            <update_rate>15</update_rate>
+            <topic>camera</topic>
+            <camera>
+                <horizontal_fov>1.05</horizontal_fov>
+                <image>
+                    <width>640</width>
+                    <height>480</height>
+                    <format>R8G8B8</format>
+                </image>
+                <clip>
+                    <near>0.1</near>
+                    <far>20.0</far>
+                </clip>
+            </camera>
+        </sensor>
+    </gazebo>
     <xacro:macro name="foot_friction" params="name">
         <gazebo reference="${name}_foot">

File: quadruped_ws/src/quadruped_description/xacro/leg.xacro (robot description, xacro)
@@ -32,19 +32,11 @@
         </joint>
         <link name="${name}_hip">
+            <!-- Visual dung cylinder don gian thay vi mesh .dae - xem ghi chu o
+                 trunk visual trong robot.xacro. Cylinder doi xung truc nen dung
+                 chung 1 origin voi collision cho ca 4 chan. -->
             <visual>
-                <xacro:if value="${(mirror_dae == True) and (front_hind_dae == True)}">
-                    <origin rpy="0 0 0" xyz="0 0 0"/>
-                </xacro:if>
-                <xacro:if value="${(mirror_dae == False) and (front_hind_dae == True)}">
-                    <origin rpy="${PI} 0 0" xyz="0 0 0"/>
-                </xacro:if>
-                <xacro:if value="${(mirror_dae == True) and (front_hind_dae == False)}">
-                    <origin rpy="0 ${PI} 0" xyz="0 0 0"/>
-                </xacro:if>
-                <xacro:if value="${(mirror_dae == False) and (front_hind_dae == False)}">
-                    <origin rpy="${PI} ${PI} 0" xyz="0 0 0"/>
-                </xacro:if>
+                <origin rpy="${PI/2.0} 0 0" xyz="0 ${hip_offset*mirror} 0"/>
                 <geometry>
-                    <mesh filename="package://quadruped_description/meshes/hip.dae" scale="1 1 1"/>
+                    <cylinder length="${hip_length}" radius="${hip_radius}"/>
                 </geometry>
             </visual>
@@ -73,13 +65,10 @@
         </joint>
         <link name="${name}_thigh">
+            <!-- Visual dung box don gian thay vi mesh .dae - xem ghi chu o trunk
+                 visual trong robot.xacro. -->
             <visual>
-                <origin rpy="0 0 0" xyz="0 0 0"/>
+                <origin rpy="0 ${PI/2.0} 0" xyz="0 0 ${-thigh_length/2.0}"/>
                 <geometry>
-                    <xacro:if value="${mirror_dae == True}">
-                        <mesh filename="package://quadruped_description/meshes/thigh.dae" scale="1 1 1"/>
-                    </xacro:if>
-                    <xacro:if value="${mirror_dae == False}">
-                        <mesh filename="package://quadruped_description/meshes/thigh_mirror.dae" scale="1 1 1"/>
-                    </xacro:if>
+                    <box size="${thigh_length} ${thigh_width} ${thigh_height}"/>
                 </geometry>
             </visual>
@@ -108,8 +97,10 @@
         </joint>
         <link name="${name}_calf">
+            <!-- Visual dung box don gian thay vi mesh .dae - xem ghi chu o trunk
+                 visual trong robot.xacro. -->
             <visual>
-                <origin rpy="0 0 0" xyz="0 0 0"/>
+                <origin rpy="0 ${PI/2.0} 0" xyz="0 0 ${-calf_length/2.0}"/>
                 <geometry>
-                    <mesh filename="package://quadruped_description/meshes/calf.dae" scale="1 1 1"/>
+                    <box size="${calf_length} ${calf_width} ${calf_height}"/>
                 </geometry>
             </visual>

File: quadruped_ws/src/quadruped_description/xacro/robot.xacro (robot description, xacro)
@@ -18,8 +18,15 @@
     <xacro:include filename="$(find quadruped_description)/xacro/gazebo.xacro"/>
     <link name="trunk">
+        <!-- Visual dung box don gian thay vi mesh .dae goc: mesh COLLADA nhieu
+             polygon (~78k faces) lam hong render context cua camera sensor tren
+             may GPU hybrid Intel+NVIDIA (da kiem chung: mesh it face render camera
+             dung, mesh nhieu face lam camera ra mau xam dong nhat - loi tang
+             gz-sim/driver). Mesh giam poly thi camera render duoc nhung nhin xau
+             hon box, nen dung box. collision/inertial giu nguyen, khong doi vat ly.
+             Xem CLAUDE.md. -->
         <visual>
             <origin rpy="0 0 0" xyz="0 0 0"/>
             <geometry>
-                <mesh filename="package://quadruped_description/meshes/base.dae" scale="1 1 1"/>
+                <box size="${trunk_length} ${trunk_width} ${trunk_height}"/>
             </geometry>
         </visual>
@@ -63,4 +70,43 @@
         </collision>
     </link>
+    <!-- Camera RGBD gan truoc trunk, dung cho track_object (xem gazebo.xacro cho sensor tag).
+         Nghieng xuong ~0.26 rad (15 deg, pitch quanh Y) de khi robot tien lai gan,
+         muc tieu duoi dat khong roi khoi khung hinh (da kiem chung: camera ngang thi
+         mat detection luc den gan vi bong tut xuong day anh). tf2 tu dong bu goc nghieng
+         nen cong thuc pinhole -> target_pose khong doi. -->
+    <joint name="camera_joint" type="fixed">
+        <parent link="trunk"/>
+        <child link="camera_link"/>
+        <origin rpy="0 0.26 0" xyz="${trunk_length/2} 0 0.02"/>
+    </joint>
+    <link name="camera_link">
+        <inertial>
+            <mass value="0.001"/>
+            <origin rpy="0 0 0" xyz="0 0 0"/>
+            <inertia ixx="0.0001" ixy="0" ixz="0" iyy="0.0001" iyz="0" izz="0.0001"/>
+        </inertial>
+        <visual>
+            <origin rpy="0 0 0" xyz="0 0 0"/>
+            <geometry>
+                <box size="0.001 0.001 0.001"/>
+            </geometry>
+        </visual>
+        <collision>
+            <origin rpy="0 0 0" xyz="0 0 0"/>
+            <geometry>
+                <box size=".001 .001 .001"/>
+            </geometry>
+        </collision>
+    </link>
+    <!-- Frame "optical" chuan REP-103 (z-forward, x-right, y-down) - cong thuc
+         pinhole trong quadruped_perception/target_pose_node.py tinh diem 3D
+         theo quy uoc nay, khac voi camera_link vat ly (x-forward giong than
+         robot) nen can xoay rieng, khong dung truc tiep camera_link. -->
+    <joint name="camera_optical_joint" type="fixed">
+        <parent link="camera_link"/>
+        <child link="camera_link_optical"/>
+        <origin rpy="${-PI/2} 0 ${-PI/2}" xyz="0 0 0"/>
+    </joint>
+    <link name="camera_link_optical"/>
     <xacro:leg name="FR" mirror="-1" mirror_dae="False" front_hind="1"  front_hind_dae="True"  />
     <xacro:leg name="FL" mirror="1"  mirror_dae="True"  front_hind="1"  front_hind_dae="True"  />

File: quadruped_ws/src/quadruped_description/xacro/ros2_control.xacro (robot description, xacro)
@@ -16,27 +16,39 @@
     <xacro:property name="standing_thigh" value="0.7894648616758762"/>
     <xacro:property name="standing_calf" value="-1.5789297233517523"/>
+    <!-- Moi khop khai bao CA HAI command_interface:
+         - position: cho baseline gait rule-based (forward_position_controller,
+           gz mo phong bang P noi bo, gain hip=100 thigh/calf=300).
+         - effort: cho RL locomotion (quadruped_rl) - node tu tinh PD torque
+           (Kp/Kd cua policy) roi gui effort truc tiep, khong dung P noi bo cua gz.
+         Chi 1 controller active moi luc (position HOAC effort), khong xung dot. -->
     <xacro:macro name="leg_ros2_control" params="name hip_gain:=100 thigh_gain:=300 calf_gain:=300">
         <joint name="${name}_hip_joint">
             <command_interface name="position"/>
+            <command_interface name="effort"/>
             <state_interface name="position">
                 <param name="initial_value">${standing_hip}</param>
             </state_interface>
             <state_interface name="velocity"/>
+            <state_interface name="effort"/>
             <param name="position_proportional_gain">${hip_gain}</param>
         </joint>
         <joint name="${name}_thigh_joint">
             <command_interface name="position"/>
+            <command_interface name="effort"/>
             <state_interface name="position">
                 <param name="initial_value">${standing_thigh}</param>
             </state_interface>
             <state_interface name="velocity"/>
+            <state_interface name="effort"/>
             <param name="position_proportional_gain">${thigh_gain}</param>
         </joint>
         <joint name="${name}_calf_joint">
             <command_interface name="position"/>
+            <command_interface name="effort"/>
             <state_interface name="position">
                 <param name="initial_value">${standing_calf}</param>
             </state_interface>
             <state_interface name="velocity"/>
+            <state_interface name="effort"/>
             <param name="position_proportional_gain">${calf_gain}</param>
         </joint>
