Commit message: Add LiDAR obstacle avoidance + SLAM navigation and MuJoCo LiDAR demos
- quadruped_navigation: reactive obstacle_avoider (LiDAR /scan -> /cmd_vel)
  with pure-logic self-test, planner, lidar_slam.launch.py (LiDAR + avoid +
  slam_toolbox map building), slam_toolbox + rviz config
- quadruped_description: add 2D LiDAR sensor (gpu_lidar) to xacro, static
  obstacles in flat_ground.sdf world
- quadruped_rl/mujoco_demo: LiDAR avoid/nav/rviz demo scripts + maze generator
- docs: LiDAR maze + pointcloud images, README/CLAUDE.md updates

File: quadruped_ws/src/quadruped_description/xacro/gazebo.xacro (robot description, xacro)
@@ -52,4 +52,34 @@
         </sensor>
     </gazebo>
+    <!-- LiDAR 2D (gpu_lidar) tren lidar_link - quet ngang 360 de ne vat can + SLAM.
+         Publish LaserScan tren /scan (bridge trong gazebo.launch.py). -->
+    <gazebo reference="lidar_link">
+        <sensor name="lidar_sensor" type="gpu_lidar">
+            <always_on>true</always_on>
+            <update_rate>10</update_rate>
+            <topic>scan</topic>
+            <gz_frame_id>lidar_link</gz_frame_id>
+            <lidar>
+                <scan>
+                    <horizontal>
+                        <samples>360</samples>
+                        <resolution>1</resolution>
+                        <min_angle>-3.14159</min_angle>
+                        <max_angle>3.14159</max_angle>
+                    </horizontal>
+                    <vertical>
+                        <samples>1</samples>
+                        <min_angle>0</min_angle>
+                        <max_angle>0</max_angle>
+                    </vertical>
+                </scan>
+                <range>
+                    <min>0.15</min>
+                    <max>8.0</max>
+                    <resolution>0.01</resolution>
+                </range>
+            </lidar>
+        </sensor>
+    </gazebo>
     <xacro:macro name="foot_friction" params="name">
         <gazebo reference="${name}_foot">

File: quadruped_ws/src/quadruped_description/xacro/robot.xacro (robot description, xacro)
@@ -109,4 +109,30 @@
     </joint>
     <link name="camera_link_optical"/>
+    <!-- LiDAR 2D gan tren noc trunk, dung cho ne vat can + SLAM (quadruped_navigation).
+         Sensor gpu_lidar khai trong gazebo.xacro, publish /scan. -->
+    <joint name="lidar_joint" type="fixed">
+        <parent link="trunk"/>
+        <child link="lidar_link"/>
+        <origin rpy="0 0 0" xyz="0.1 0 0.09"/>
+    </joint>
+    <link name="lidar_link">
+        <inertial>
+            <mass value="0.001"/>
+            <origin rpy="0 0 0" xyz="0 0 0"/>
+            <inertia ixx="0.0001" ixy="0" ixz="0" iyy="0.0001" iyz="0" izz="0.0001"/>
+        </inertial>
+        <visual>
+            <origin rpy="0 0 0" xyz="0 0 0"/>
+            <geometry>
+                <cylinder radius="0.035" length="0.04"/>
+            </geometry>
+        </visual>
+        <collision>
+            <origin rpy="0 0 0" xyz="0 0 0"/>
+            <geometry>
+                <cylinder radius="0.035" length="0.04"/>
+            </geometry>
+        </collision>
+    </link>
     <xacro:leg name="FR" mirror="-1" mirror_dae="False" front_hind="1"  front_hind_dae="True"  />
     <xacro:leg name="FL" mirror="1"  mirror_dae="True"  front_hind="1"  front_hind_dae="True"  />
